File: Design an RP2040 board with KiCad/Chapter 5/rp2040_board/rp2040_board.kicad_sch (KiCad schematic)
At the start: 30 parts, among them J1 USB_B_Micro, J2 Conn_01x02, J3 Conn_02x18_Odd_Even, J4 Conn_02x18_Odd_Even, U1 NCP1117-3.3_SOT223, U2 W25Q128JVS, U3 RP2040, Y1 Crystal_GND23

Commit message: Small improvements for RP2040 board
Parts:
- added H1, H2, H3, H4: MountingHole, MountingHole:MountingHole_2.7mm_M2.5, symbol Mechanical:MountingHole
