File: rp2350a_board/rp2350a_board/rp2350a_board.kicad_sch (KiCad schematic)
At the start: 44 parts, among them J1 USB_B_Micro, J2 Conn_02x18_Odd_Even, J3 Conn_02x18_Odd_Even, J4 SM03B-SRSS-TB, SW1 SW_Push, SW2 SW_Push, U1 RP2350_60QFN, U2 NCP1117-3.3_SOT223, U3 W25Q128JVS, Y1 Crystal_GND24

Commit message: Some fixes in schematic
Parts:
- removed C20, C21: 100n, symbol Device:C
- added R2: 1k, symbol Device:R
- R6: value 5k -> 1k
- U1: footprint RP2350_60QFN_minimal:RP2350-QFN-60-1EP_7x7_P0.4mm_EP3.4x3.4mm_ThermalVias -> Package_DFN_QFN:QFN-60-1EP_7x7mm_P0.4mm_EP3.4x3.4mm_ThermalVias
Connections:
- net +3V3 is gone; now on net +1V1: C12.1, C13.1, C14.1, C15.1, C16.1, C17.1, C18.1, C19.1, C2.1, C5.1, C6.1, J2.2 (Pin_2), R1.1, R3.1, U1.1 (IOVDD), U1.11 (IOVDD), U1.20 (IOVDD), U1.30 (IOVDD), U1.38 (IOVDD), U1.44 (ADC_AVDD), U1.45 (IOVDD), U1.49 (VREG_VIN), U1.53 (USB_OTP_VDD), U1.54 (QSPI_IOVDD), U2.2 (VO), U3.8 (VCC)
- net XOUT: now also R2.2; no longer C4.2, Y1.3
- new net: C4.2, R2.1, Y1.3
Changed lines of the file:
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@@
 	)
 	(junction
-		(at 264.16 24.13)
-		(diameter 0)
-		(color 0 0 0 0)
-	)
-	(junction
 		(at 224.79 91.44)
 		(diameter 0)
@@
 	)
 	(junction
-		(at 275.59 31.75)
-		(diameter 0)
-		(color 0 0 0 0)
-	)
-	(junction
 		(at 224.79 121.92)
 		(diameter 0)
@@
 	(wire
 		(pts
-			(xy 264.16 24.13) (xy 275.59 24.13)
+			(xy 252.73 24.13) (xy 264.16 24.13)
 		)
 		(stroke
@@
 	(wire
 		(pts
-			(xy 77.47 158.75) (xy 99.06 158.75)
+			(xy 46.99 121.92) (xy 60.96 121.92)
 		)
 		(stroke
@@
 	(wire
 		(pts
-			(xy 46.99 121.92) (xy 60.96 121.92)
+			(xy 90.17 77.47) (xy 128.27 77.47)
 		)
 		(stroke
@@
 	(wire
 		(pts
-			(xy 90.17 77.47) (xy 128.27 77.47)
+			(xy 224.79 124.46) (xy 224.79 121.92)
 		)
 		(stroke
@@
 	(wire
 		(pts
-			(xy 224.79 124.46) (xy 224.79 121.92)
+			(xy 251.46 114.3) (xy 264.16 114.3)
 		)
 		(stroke
@@
 	(wire
 		(pts
-			(xy 251.46 114.3) (xy 264.16 114.3)
+			(xy 224.79 86.36) (xy 224.79 88.9)
 		)
 		(stroke
@@
 	(wire
 		(pts
-			(xy 224.79 86.36) (xy 224.79 88.9)
+			(xy 264.16 24.13) (xy 264.16 31.75)
 		)
 		(stroke
@@
 	(wire
 		(pts
-			(xy 275.59 31.75) (xy 275.59 35.56)
+			(xy 264.16 31.75) (xy 264.16 35.56)
 		)
 		(stroke
@@
 	(wire
 		(pts
-			(xy 264.16 31.75) (xy 275.59 31.75)
+			(xy 252.73 31.75) (xy 264.16 31.75)
 		)
 		(stroke
@@
 	(wire
 		(pts
-			(xy 252.73 24.13) (xy 264.16 24.13)
-		)
-		(stroke
-			(width 0)
-			(type default)
-		)
-	)
-	(wire
-		(pts
 			(xy 251.46 91.44) (xy 264.16 91.44)
 		)
@@
 	(wire
 		(pts
-			(xy 252.73 31.75) (xy 264.16 31.75)
-		)
-		(stroke
-			(width 0)
-			(type default)
-		)
-	)
-	(wire
-		(pts
 			(xy 93.98 127) (xy 90.17 127)
 		)
@@
 	(wire
 		(pts
+			(xy 95.25 158.75) (xy 104.14 158.75)
+		)
+		(stroke
+			(width 0)
+			(type default)
+		)
+	)
+	(wire
+		(pts
 			(xy 127 31.75) (xy 137.16 31.75)
 		)
@@
 	(wire
 		(pts
-			(xy 77.47 151.13) (xy 99.06 151.13)
+			(xy 77.47 151.13) (xy 104.14 151.13)
 		)
 		(stroke
@@
 	(wire
 		(pts
+			(xy 87.63 158.75) (xy 77.47 158.75)
+		)
+		(stroke
+			(width 0)
+			(type default)
+		)
+	)
+	(wire
+		(pts
 			(xy 237.49 99.06) (xy 245.11 99.06)
 		)
@@
 	)
 	(label "XIN"
-		(at 99.06 151.13 180)
+		(at 104.14 151.13 180)
 		(effects
 			(font
@@
 	)
 	(label "XOUT"
-		(at 99.06 158.75 180)
+		(at 104.14 158.75 180)
 		(effects
 			(font
@@
 	(symbol
 		(lib_id "power:GND")
-		(at 275.59 35.56 0)
+		(at 264.16 35.56 0)
 		(unit 1)
 		(exclude_from_sim no)
@@
 		(fields_autoplaced yes)
 		(property "Reference" "#PWR014"
-			(at 275.59 41.91 0)
+			(at 264.16 41.91 0)
 			(effects
 				(font
@@
 		)
 		(property "Value" "GND"
-			(at 275.59 40.64 0)
+			(at 264.16 40.64 0)
 			(effects
 				(font
@@
 		)
 		(property "Footprint" ""
-			(at 275.59 35.56 0)
+			(at 264.16 35.56 0)
 			(effects
 				(font
@@
 		)
 		(property "Datasheet" ""
-			(at 275.59 35.56 0)
+			(at 264.16 35.56 0)
 			(effects
 				(font
@@
 		)
 		(property "Description" "Power symbol creates a global label with name \"GND\" , ground"
-			(at 275.59 35.56 0)
+			(at 264.16 35.56 0)
 			(effects
 				(font
@@
 	)
 	(symbol
-		(lib_id "Device:C")
-		(at 275.59 27.94 0)
+		(lib_id "Device:R")
+		(at 91.44 158.75 90)
 		(unit 1)
 		(exclude_from_sim no)
@@
 		(on_board yes)
 		(dnp no)
-		(fields_autoplaced yes)
-		(property "Reference" "C21"
-			(at 279.4 26.6699 0)
+		(property "Reference" "R2"
+			(at 93.218 153.924 90)
 			(effects
 				(font
 					(size 1.27 1.27)
 				)
-				(justify left)
 			)
 		)
-		(property "Value" "100n"
-			(at 279.4 29.2099 0)
+		(property "Value" "1k"
+			(at 93.218 156.464 90)
 			(effects
 				(font
 					(size 1.27 1.27)
 				)
-				(justify left)
 			)
 		)
 		(property "Footprint" ""
-			(at 276.5552 31.75 0)
+			(at 91.44 160.528 90)
 			(effects
 				(font
@@
 		)
 		(property "Datasheet" "~"
-			(at 275.59 27.94 0)
+			(at 91.44 158.75 0)
 			(effects
 				(font
@@
 			)
 		)
-		(property "Description" "Unpolarized capacitor"
-			(at 275.59 27.94 0)
+		(property "Description" "Resistor"
+			(at 91.44 158.75 0)
 			(effects
 				(font
@@
 			)
 		)
-		(pin "1"
-		)
 		(pin "2"
 		)
+		(pin "1"
+		)
 		(instances
-			(project "rp2354a_board"
+			(project ""
 				(path "/4801170d-1806-4299-a78b-2cb59e31934d"
-					(reference "C21")
+					(reference "R2")
 					(unit 1)
 				)
@@
 			)
 		)
-		(property "Value" "5k"
+		(property "Value" "1k"
 			(at 109.22 81.28 90)
 			(effects
@@
 			)
 		)
-		(property "Footprint" "RP2350_60QFN_minimal:RP2350-QFN-60-1EP_7x7_P0.4mm_EP3.4x3.4mm_ThermalVias"
+		(property "Footprint" "Package_DFN_QFN:QFN-60-1EP_7x7mm_P0.4mm_EP3.4x3.4mm_ThermalVias"
 			(at 140.97 106.68 0)
 			(effects
@@
 					(unit 1)
 				)
-			)
-		)
-	)
-	(symbol
-		(lib_id "Device:C")
-		(at 264.16 27.94 0)
-		(unit 1)
-		(exclude_from_sim no)
-		(in_bom yes)
-		(on_board yes)
-		(dnp no)
-		(fields_autoplaced yes)
-		(property "Reference" "C20"
-			(at 267.97 26.6699 0)
-			(effects
-				(font
-					(size 1.27 1.27)
-				)
-				(justify left)
-			)
-		)
-		(property "Value" "100n"
-			(at 267.97 29.2099 0)
-			(effects
-				(font
-					(size 1.27 1.27)
-				)
-				(justify left)
-			)
-		)
-		(property "Footprint" ""
-			(at 265.1252 31.75 0)
-			(effects
-				(font
-					(size 1.27 1.27)
-				)
-				(hide yes)
-			)
-		)
-		(property "Datasheet" "~"
-			(at 264.16 27.94 0)
-			(effects
-				(font
-					(size 1.27 1.27)
-				)
-				(hide yes)
-			)
-		)
-		(property "Description" "Unpolarized capacitor"
-			(at 264.16 27.94 0)
-			(effects
-				(font
-					(size 1.27 1.27)
-				)
-				(hide yes)
-			)
-		)
-		(pin "1"
-		)
-		(pin "2"
-		)
-		(instances
-			(project "rp2354a_board"
-				(path "/4801170d-1806-4299-a78b-2cb59e31934d"
-					(reference "C20")
-					(unit 1)
-				)

Commit message: Finish assignment of footprints
Parts:
- C1, C19, C5: footprint (none) -> Capacitor_SMD:C_0805_2012Metric
- C10, C11, C12, C13, C14, C15, C16, C17, C18, C2, C3, C4, C8, C9: footprint (none) -> Capacitor_SMD:C_0402_1005Metric
- C6, C7: footprint (none) -> RP2350_60QFN_minimal:C_0402_1005Metric_small_pads
- J1: footprint (none) -> Connector_USB:USB_Micro-B_Amphenol_10103594-0001LF_Horizontal
- J2, J3: footprint (none) -> Connector_PinHeader_2.54mm:PinHeader_2x18_P2.54mm_Vertical
- L1: footprint (none) -> RP2350_60QFN_minimal:L_pol_2016
- R1, R10, R2, R6, R7, R8, R9: footprint (none) -> Resistor_SMD:R_0402_1005Metric
- R4: value 1K -> 1k; footprint (none) -> Resistor_SMD:R_0402_1005Metric
- R5: renamed from R3; footprint (none) -> Resistor_SMD:R_0402_1005Metric
- SW1, SW2: footprint (none) -> Button_Switch_SMD:SW_Push_1P1T_NO_Vertical_Wuerth_434133025816
- Y1: value Crystal_GND24 -> ABM8-272-T3; footprint (none) -> Crystal:Crystal_SMD_3225-4Pin_3.2x2.5mm
Changed lines of the file:
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@@
 			)
 		)
-		(property "Footprint" ""
+		(property "Footprint" "Capacitor_SMD:C_0402_1005Metric"
 			(at 67.31 150.1648 0)
 			(effects
@@
 			)
 		)
-		(property "Footprint" ""
+		(property "Footprint" "Capacitor_SMD:C_0402_1005Metric"
 			(at 127.9652 31.75 0)
 			(effects
@@
 			)
 		)
-		(property "Footprint" ""
+		(property "Footprint" "Button_Switch_SMD:SW_Push_1P1T_NO_Vertical_Wuerth_434133025816"
 			(at 87.63 91.44 0)
 			(effects
@@
 			)
 		)
-		(property "Footprint" ""
+		(property "Footprint" "RP2350_60QFN_minimal:C_0402_1005Metric_small_pads"
 			(at 79.7052 71.12 0)
 			(effects
@@
 			)
 		)
-		(property "Value" "1K"
+		(property "Value" "1k"
 			(at 97.79 123.19 90)
 			(effects
@@
 			)
 		)
-		(property "Footprint" ""
+		(property "Footprint" "Resistor_SMD:R_0402_1005Metric"
 			(at 97.79 128.778 90)
 			(effects
@@
 			)
 		)
-		(property "Footprint" ""
+		(property "Footprint" "Capacitor_SMD:C_0402_1005Metric"
 			(at 253.6952 31.75 0)
 			(effects
@@
 			)
 		)
-		(property "Value" "Crystal_GND24"
+		(property "Value" "ABM8-272-T3"
 			(at 77.216 148.082 90)
 			(effects
@@
 			)
 		)
-		(property "Footprint" ""
+		(property "Footprint" "Crystal:Crystal_SMD_3225-4Pin_3.2x2.5mm"
 			(at 77.47 154.94 0)
 			(effects
@@
 			)
 		)
-		(property "Footprint" ""
+		(property "Footprint" "Resistor_SMD:R_0402_1005Metric"
 			(at 45.212 113.03 90)
 			(effects
@@
 			)
 		)
-		(property "Footprint" ""
+		(property "Footprint" "Capacitor_SMD:C_0805_2012Metric"
 			(at 213.0552 105.41 0)
 			(effects
@@
 			)
 		)
-		(property "Footprint" ""
+		(property "Footprint" "Connector_USB:USB_Micro-B_Amphenol_10103594-0001LF_Horizontal"
 			(at 25.4 26.67 0)
 			(effects
@@
 			)
 		)
-		(property "Footprint" ""
+		(property "Footprint" "Capacitor_SMD:C_0402_1005Metric"
 			(at 105.1052 31.75 0)
 			(effects
@@
 			)
 		)
-		(property "Footprint" ""
+		(property "Footprint" "Capacitor_SMD:C_0402_1005Metric"
 			(at 113.9952 58.42 0)
 			(effects
@@
 			)
 		)
-		(property "Footprint" ""
+		(property "Footprint" "Capacitor_SMD:C_0805_2012Metric"
 			(at 80.9752 30.48 0)
 			(effects
@@
 			)
 		)
-		(property "Footprint" ""
+		(property "Footprint" "Capacitor_SMD:C_0402_1005Metric"
 			(at 185.1152 31.75 0)
 			(effects
@@
 			)
 		)
-		(property "Footprint" ""
+		(property "Footprint" "Capacitor_SMD:C_0402_1005Metric"
 			(at 28.9052 111.76 0)
 			(effects
@@
 			)
 		)
-		(property "Footprint" ""
+		(property "Footprint" "Resistor_SMD:R_0402_1005Metric"
 			(at 66.04 114.808 90)
 			(effects
@@
 			)
 		)
-		(property "Footprint" ""
+		(property "Footprint" "Resistor_SMD:R_0402_1005Metric"
 			(at 91.44 160.528 90)
 			(effects
@@
 			)
 		)
-		(property "Footprint" ""
+		(property "Footprint" "Capacitor_SMD:C_0402_1005Metric"
 			(at 196.5452 31.75 0)
 			(effects
@@
 			)
 		)
-		(property "Footprint" ""
+		(property "Footprint" "Capacitor_SMD:C_0402_1005Metric"
 			(at 207.9752 31.75 0)
 			(effects
@@
 			)
 		)
-		(property "Footprint" ""
+		(property "Footprint" "Connector_PinHeader_2.54mm:PinHeader_2x18_P2.54mm_Vertical"
 			(at 269.24 106.68 0)
 			(effects
@@
 			)
 		)
-		(property "Footprint" ""
+		(property "Footprint" "Capacitor_SMD:C_0402_1005Metric"
 			(at 67.31 157.7848 0)
 			(effects
@@
 			)
 		)
-		(property "Footprint" ""
+		(property "Footprint" "Resistor_SMD:R_0402_1005Metric"
 			(at 203.2 67.818 90)
 			(effects
@@
 			)
 		)
-		(property "Footprint" ""
+		(property "Footprint" "Capacitor_SMD:C_0402_1005Metric"
 			(at 116.5352 31.75 0)
 			(effects
@@
 			)
 		)
-		(property "Footprint" ""
+		(property "Footprint" "Capacitor_SMD:C_0805_2012Metric"
 			(at 46.6852 30.48 0)
 			(effects
@@
 			)
 		)
-		(property "Footprint" ""
+		(property "Footprint" "Button_Switch_SMD:SW_Push_1P1T_NO_Vertical_Wuerth_434133025816"
 			(at 109.22 121.92 0)
 			(effects
@@
 			)
 		)
-		(property "Footprint" ""
+		(property "Footprint" "Resistor_SMD:R_0402_1005Metric"
 			(at 203.2 60.198 90)
 			(effects
@@
 			)
 		)
-		(property "Footprint" ""
+		(property "Footprint" "Connector_PinHeader_2.54mm:PinHeader_2x18_P2.54mm_Vertical"
 			(at 229.87 106.68 0)
 			(effects
@@
 			)
 		)
-		(property "Footprint" ""
+		(property "Footprint" "RP2350_60QFN_minimal:C_0402_1005Metric_small_pads"
 			(at 91.1352 71.12 0)
 			(effects
@@
 			)
 		)
-		(property "Footprint" ""
+		(property "Footprint" "Resistor_SMD:R_0402_1005Metric"
 			(at 109.22 86.868 90)
 			(effects
@@
 			)
 		)
-		(property "Footprint" ""
+		(property "Footprint" "Capacitor_SMD:C_0402_1005Metric"
 			(at 242.2652 31.75 0)
 			(effects
@@
 			)
 		)
-		(property "Footprint" ""
+		(property "Footprint" "Resistor_SMD:R_0402_1005Metric"
 			(at 66.04 123.698 90)
 			(effects
@@
 			)
 		)
-		(property "Footprint" ""
+		(property "Footprint" "Capacitor_SMD:C_0402_1005Metric"
 			(at 230.8352 31.75 0)
 			(effects
@@
 			)
 		)
-		(property "Footprint" ""
+		(property "Footprint" "RP2350_60QFN_minimal:L_pol_2016"
 			(at 99.06 67.31 0)
 			(effects
@@
 		(dnp no)
 		(fields_autoplaced yes)
-		(property "Reference" "R3"
+		(property "Reference" "R5"
 			(at 104.14 44.45 90)
 			(effects
@@
 			)
 		)
-		(property "Footprint" ""
+		(property "Footprint" "Resistor_SMD:R_0402_1005Metric"
 			(at 104.14 52.578 90)
 			(effects
@@
 			(project ""
 				(path "/4801170d-1806-4299-a78b-2cb59e31934d"
-					(reference "R3")
+					(reference "R5")
 					(unit 1)
 				)
@@
 			)
 		)
-		(property "Footprint" ""
+		(property "Footprint" "Capacitor_SMD:C_0402_1005Metric"
 			(at 219.4052 31.75 0)
 			(effects
